File: camera.kicad_sch (KiCad schematic)
At the start: 1 part, among them U1 K230_Rewired

Commit message: a lot of stuff happened
Parts:
- removed U1: K230_Rewired, footprints:BGA-390_L13.0-W13.0-P0.65-TL_C9900054646, symbol LCSC:K230_Rewired
- added U1: K230_Rewired, footprints:BGA-390_L13.0-W13.0-P0.65-TL_C9900054646, symbol LCSC:K230_Rewired
- added U3: HC-FPC-0_5-22P-CXH20, footprints:FPC-SMD_22P-P0.50_HC-FPC-0.5-22P-CXH20, symbol LCSC:HC-FPC-0_5-22P-CXH20
Other:
- removed sheet Camera
- removed sheet GPIO
- removed sheet Power
- removed sheet RAM
- removed sheet Storage
