File: gpio.kicad_sch (KiCad schematic)
At the start: 1 part, among them U1 K230_Rewired

Commit message: a lot of stuff happened
Parts:
- removed U1: K230_Rewired, footprints:BGA-390_L13.0-W13.0-P0.65-TL_C9900054646, symbol LCSC:K230_Rewired
- added D1: LED, LED_SMD:LED_PLCC_2835, symbol Device:LED
- added J1, J2: REV_JST_SMD, Custom:JST_SH_SM04B-SRSS-TB_1x04-1MP_P1.00mm_Horizontal, symbol Custom:REV_JST_SMD
- added U1: K230_Rewired, footprints:BGA-390_L13.0-W13.0-P0.65-TL_C9900054646, symbol LCSC:K230_Rewired
Other:
- removed sheet Camera
- removed sheet GPIO
- removed sheet Power
- removed sheet RAM
- removed sheet Storage
