File: power.kicad_sch (KiCad schematic)
At the start: 1 part, among them U1 K230_Rewired

Commit message: a lot of stuff happened
Parts:
- removed U1: K230_Rewired, footprints:BGA-390_L13.0-W13.0-P0.65-TL_C9900054646, symbol LCSC:K230_Rewired
- added U1: K230_Rewired, footprints:BGA-390_L13.0-W13.0-P0.65-TL_C9900054646, symbol LCSC:K230_Rewired
- added U5: RT9992ZQW, Package_DFN_QFN:Texas_RSN_WQFN-32-1EP_4x4mm_P0.4mm_EP2.8x2.8mm, symbol LCSC:RT9992ZQW
Connections:
- new net: U1.A16 (VSS), U1.L15 (VSS)
- new net: U1.C13 (VSS), U1.N12 (VSS)
- new net: U1.E12 (VSS), U1.R12 (VSS)
- new net: U1.E14 (VSS), U1.R14 (VSS)
- new net: U1.E16 (VSS), U1.R16 (VSS)
Other:
- removed sheet Camera
- removed sheet GPIO
- removed sheet Power
- removed sheet RAM
- removed sheet Storage
