File: storage.kicad_sch (KiCad schematic)
At the start: 1 part, among them U1 K230_Rewired

Commit message: a lot of stuff happened
Parts:
- removed U1: K230_Rewired, footprints:BGA-390_L13.0-W13.0-P0.65-TL_C9900054646, symbol LCSC:K230_Rewired
- added U1: K230_Rewired, footprints:BGA-390_L13.0-W13.0-P0.65-TL_C9900054646, symbol LCSC:K230_Rewired
- added U2: ZDSD04GLGEAG, footprints:LGA-8_L8.0-W6.0-P1.27-TL-1, symbol LCSC:ZDSD04GLGEAG
Connections:
- new net: U1.P1 (SDIO_D2), U2.1 (DAT2)
- new net: U1.P2 (SDIO_D3), U2.2 (DAT3)
- new net: U1.N2 (SDIO_CLK), U2.3 (CLK)
- new net: U1.M2 (SDIO_CMD), U2.5 (CMD)
- new net: U1.P3 (SDIO_D0), U2.6 (DAT0)
- new net: U1.N1 (SDIO_D1), U2.7 (DAT1)
Other:
- removed sheet Camera
- removed sheet GPIO
- removed sheet Power
- removed sheet RAM
- removed sheet Storage
