File: untitled.kicad_sch (KiCad schematic)
At the start: 1 part, among them U1 K230_Rewired

Commit message: a lot of stuff happened
Parts:
- removed U1: K230_Rewired, footprints:BGA-390_L13.0-W13.0-P0.65-TL_C9900054646, symbol LCSC:K230_Rewired
- added U1: K230_Rewired, footprints:BGA-390_L13.0-W13.0-P0.65-TL_C9900054646, symbol LCSC:K230_Rewired
- added U4: K4E8E324ED-EGCG, footprints:BGA-178_L11.5W11.0-P0.65-TL, symbol LCSC:K4E8E324ED-EGCG
Connections:
- new net: U1.U17 (DDR_DQ29_DQA7), U4.B10 (DQ29)
- new net: U1.Y18 (DDR_DQ28_DQA6), U4.B11 (DQ28)
- new net: U1.U16 (DDR_DQ31_DQA0), U4.B8 (DQ31)
- new net: U1.T16 (DDR_DQ30_DQA1), U4.B9 (DQ30)
- new net: U1.V18 (DDR_DQ25_DQA5), U4.C10 (DQ25)
- new net: U1.W18 (DDR_DQ24_DQA4), U4.C11 (DQ24)
- new net: U1.Y16 (DDR_DQ27_DQA3), U4.C8 (DQ27)
- new net: U1.V16 (DDR_DQ26_DQA2), U4.C9 (DQ26)
- new net: U1.T17 (DDR_DQ15_DQA15), U4.D9 (DQ15)
- new net: U1.U20 (DDR_DQ13_DQA11), U4.E10 (DQ13)
- new net: U1.T18 (DDR_DQ12_DQA9), U4.E11 (DQ12)
- new net: U1.U18 (DDR_DQ14_DQA13), U4.E9 (DQ14)
- new net: U1.P16 (DDR_DQ9_DQA14), U4.F10 (DQ9)
- new net: U1.R18 (DDR_DQ8_DQA10), U4.F11 (DQ8)
- new net: U1.W19 (DDR_DQ11_DQA12), U4.F8 (DQ11)
- new net: U1.R17 (DDR_DQ10_DQA8), U4.F9 (DQ10)
- new net: U1.B19 (DDR_DQ6_DQB7), U4.M10 (DQ6)
- new net: U1.C19 (DDR_DQ7_DQB6), U4.M11 (DQ7)
- new net: U1.E18 (DDR_DQ4_DQB2), U4.M8 (DQ4)
- new net: U1.E17 (DDR_DQ5_DQB3), U4.M9 (DQ5)
- new net: U1.D17 (DDR_DQ2_DQB0), U4.N10 (DQ2)
- new net: U1.C18 (DDR_DQ3_DQB5), U4.N11 (DQ3)
- new net: U1.D16 (DDR_DQ1_DQB1), U4.N9 (DQ1)
- new net: U1.C17 (DDR_DQ0_DQB4), U4.P9 (DQ0)
- new net: U1.B17 (DDR_DQ22_DQB12), U4.R10 (DQ22)
- new net: U1.B16 (DDR_DQ23_DQB15), U4.R11 (DQ23)
- new net: U1.D14 (DDR_DQ20_DQB8), U4.R8 (DQ20)
- new net: U1.A14 (DDR_DQ21_DQB9), U4.R9 (DQ21)
- new net: U1.C16 (DDR_DQ18_DQB13), U4.T10 (DQ18)
- new net: U1.A17 (DDR_DQ19_DQB14), U4.T11 (DQ19)
- new net: U1.C14 (DDR_DQ16_DQB11), U4.T8 (DQ16)
- new net: U1.B14 (DDR_DQ17_DQB10), U4.T9 (DQ17)
- new net DDR.CA0: U1.K20 (DDR_CA0_NC), U4.R2 (CA0)
- new net DDR.CA1: U1.L20 (DDR_CA1_NC), U4.P2 (CA1)
- new net DDR.CA2: U1.M20 (DDR_CA2_NA), U4.N2 (CA2)
- new net DDR.CA3: U1.L17 (DDR_CA3_NC), U4.N3 (CA3)
- new net DDR.CA4: U1.M19 (DDR_CA4_CAA0), U4.M3 (CA4)
- new net DDR.CA5: U1.L16 (DDR_CA5_CAA1), U4.F3 (CA5)
- new net DDR.CA6: U1.N19 (DDR_CA6_CAA2), U4.E3 (CA6)
- new net DDR.CA7: U1.N20 (DDR_CA7_CAA3), U4.E2 (CA7)
- new net DDR.CA8: U1.M18 (DDR_CA8_CAA4), U4.D2 (CA8)
- new net DDR.CA9: U1.P19 (DDR_CA9_CAA5), U4.C2 (CA9)
- new net DDR.DM0: U1.D18 (DDR_DM0_DMIB0), U4.L8 (DM0)
- new net DDR.DM1: U1.P17 (DDR_DM1_DMIA1), U4.G8 (DM1)
- new net DDR.DM2: U1.C15 (DDR_DM2_DMIB1), U4.P8 (DM2)
- new net DDR.DM3: U1.V17 (DDR_DM3_DMIA0), U4.D8 (DM3)
- new net DDR.DQS_N0: U1.A18 (DDR_DQS0N_DQSB0N), U4.L11 (DQS0_c)
- new net DDR.DQS_N1: U1.V19 (DDR_DQS1N_DQSA1N), U4.G11 (DQS1_c)
- new net DDR.DQS_N2: U1.A15 (DDR_DQS2N_DQSB1N), U4.P11 (DQS2_c)
- new net DDR.DQS_N3: U1.Y17 (DDR_DQS3N_DQSA0N), U4.D11 (DQS3_c)
- new net DDR.DQS_P0: U1.B18 (DDR_DQS0P_DQSB0P), U4.L10 (DQS0_t)
- new net DDR.DQS_P1: U1.V20 (DDR_DQS1P_DQSA1P), U4.G10 (DQS1_t)
- new net DDR.DQS_P2: U1.B15 (DDR_DQS2P_DQSB1P), U4.P10 (DQS2_t)
- new net DDR.DQS_P3: U1.W17 (DDR_DQS3P_DQSA0P), U4.D10 (DQS3_t)
Other:
- removed sheet Camera
- removed sheet GPIO
- removed sheet Power
- removed sheet RAM
- removed sheet Storage
