File: KiCAD Files/untitled.kicad_sch (KiCad schematic)
At the start: 2 parts, among them U1 K230_Rewired, U4 K4E8E324ED-EGCG

Commit message: added ram and flash
Parts:
- added C1, C2: 100nF, Capacitor_SMD:C_0402_1005Metric, symbol Device:C
- added C10, C11, C12, C13, C14, C15, C16, C17, C18, C19, C20, C21, C22, C23, C24, C27, C28, C29, C30, C31, C32, C33, C34, C5, C8, C9: 100nF, symbol Device:C
- added C25, C3, C6: 22uF, symbol Device:C
- added C26, C4, C7: 4.7uF, symbol Device:C
- added NT1: NetTie_2, symbol Device:NetTie_2
- added NT2: NetTie_4, symbol Device:NetTie_4
- added R1, R2: 240R, symbol Device:R
- added R10, R11, R12, R13, R14, R15, R16, R17, R18, R19, R20, R21, R22, R23, R24, R25, R26, R27, R28, R29, R3, R30, R31, R32, R33, R34, R35, R4, R5, R6, R7, R8, R9: 120R, PCM_Resistor_SMD_AKL:R_0402_1005Metric, symbol Device:R
- added R36: 240R, PCM_Resistor_SMD_AKL:R_0402_1005Metric, symbol Device:R
Connections:
- net DDR.CA0: now also R13.2, R14.1
- net DDR.CA1: now also R15.2, R16.1
- net DDR.CA2: now also R17.2, R18.1
- net DDR.CA3: now also R19.2, R20.1
- net DDR.CA4: now also R21.2, R22.1
- net DDR.CA5: now also R23.2, R24.1
- net DDR.CA6: now also R25.2, R26.1
- net DDR.CA7: now also R27.2, R28.1
- net DDR.CA8: now also R29.2, R30.1
- net DDR.CA9: now also R31.2, R32.1
- net DDR_VDD1: now reaches U4.A10 (VDD1)
- net DDR_VDD1: now also U4.A3 (VDD1), U4.A4 (VDD1), U4.A5 (VDD1), U4.A6 (VDD1), U4.U10 (VDD1), U4.U3 (VDD1), U4.U4 (VDD1), U4.U5 (VDD1), U4.U6 (VDD1), C25.1, C26.1, C29.1, C30.1, C31.1, C32.1, C33.1, C34.1, NT1.2
- net DDR_VDDQ: now reaches U4.A11 (VDDQ)
- net DDR_VDDQ: now also U4.C12 (VDDQ), U4.E12 (VDDQ), U4.E8 (VDDQ), U4.G12 (VDDQ), U4.H11 (VDDQ), U4.H8 (VDDQ), U4.H9 (VDDQ), U4.J10 (VDDQ), U4.J9 (VDDQ), U4.K11 (VDDQ), U4.K8 (VDDQ), U4.L12 (VDDQ), U4.N12 (VDDQ), U4.N8 (VDDQ), U4.R12 (VDDQ), U4.U11 (VDDQ), C10.1, C11.1, C12.1, C13.1, C14.1, C15.1, C16.1, C17.1, C18.1, C19.1, C20.1, C21.1, C22.1, C23.1, C24.1, C27.1, C28.1, C3.1, C4.1, C5.1, C6.1, C7.1, C8.1, C9.1, NT2.4, R11.1, R13.1, R15.1, R17.1, R19.1, R21.1, R23.1, R25.1, R27.1, R29.1, R3.1, R31.1, R33.1, R35.1, R5.1, R7.1, R9.1
- net DDR_VDD2: now reaches U4.A8 (VDD2)
- net DDR_VDD2: now also U4.A9 (VDD2), U4.D4 (VDD2), U4.D5 (VDD2), U4.D6 (VDD2), U4.G5 (VDD2), U4.H12 (VDD2), U4.H5 (VDD2), U4.H6 (VDD2), U4.J5 (VDD2), U4.J6 (VDD2), U4.K12 (VDD2), U4.K5 (VDD2), U4.K6 (VDD2), U4.L5 (VDD2), U4.P4 (VDD2), U4.P5 (VDD2), U4.P6 (VDD2), U4.U8 (VDD2), U4.U9 (VDD2), NT2.2
- net GND: now reaches U4.B12 (VSSQ)
- net GND: now also U4.B2 (VSS), U4.B5 (VSS), U4.B6 (VSSQ), U4.C3 (VSSCA), U4.C5 (VSS), U4.C6 (VSSQ), U4.D12 (VSSQ), U4.D3 (VSSCA), U4.E4 (VSS), U4.E5 (VSS), U4.E6 (VSSQ), U4.F12 (VSSQ), U4.F4 (VSSCA), U4.F5 (VSS), U4.F6 (VSSQ), U4.G3 (VSSCA), U4.G4 (VSSCA), U4.G6 (VSSQ), U4.G9 (VSSQ), U4.H10 (VSSQ), U4.H2 (VSS), U4.J12 (VSS), U4.J4 (VSSCA), U4.K10 (VSSQ), U4.K2 (VSS), U4.L6 (VSS), U4.L9 (VSSQ), U4.M12 (VSSQ), U4.M4 (VSSCA), U4.M5 (VSSCA), U4.M6 (VSSQ), U4.N4 (VSS), U4.N5 (VSS), U4.N6 (VSSQ), U4.P12 (VSSQ), U4.P3 (VSSCA), U4.R4 (VSS), U4.R5 (VSS), U4.R6 (VSSQ), U4.T12 (VSSQ), U4.T2 (VSS), U4.T3 (VSS), U4.T4 (VSS), U4.T5 (VSS), U4.T6 (VSSQ), C1.2, C10.2, C11.2, C12.2, C13.2, C14.2, C15.2, C16.2, C17.2, C18.2, C19.2, C2.2, C20.2, C21.2, C22.2, C23.2, C24.2, C25.2, C26.2, C27.2, C28.2, C29.2, C3.2, C30.2, C31.2, C32.2, C33.2, C34.2, C4.2, C5.2, C6.2, C7.2, C8.2, C9.2, R1.2, R10.2, R12.2, R14.2, R16.2, R18.2, R2.2, R20.2, R22.2, R24.2, R26.2, R28.2, R30.2, R32.2, R34.2, R36.2, R4.2, R6.2, R8.2
- net at U4.B3 (ZQ): now also R2.1
- net DDR_VDDCA: now reaches U4.F2 (VDDCA)
- net DDR_VDDCA: now also U4.G2 (VDDCA), U4.H3 (VDDCA), U4.L2 (VDDCA), U4.M2 (VDDCA), NT2.3
- net DDR.VREF_CA: now reaches U4.H4 (VRef(CA))
- net DDR.VREF_CA: now also C1.1, R33.2, R34.1
- net DDR.VREF_DQ: now reaches U4.J11 (VRef(DQ))
- net DDR.VREF_DQ: now also C2.1, R35.2, R36.1
- net DDR_CK-: now reaches U4.J2 (CK_N)
- net DDR_CK-: now also U1.R20 (DDR_CKN_CKAN), R5.2, R6.1
- net DDR_CK+: now reaches U4.J3 (CK_P)
- net DDR_CK+: now also U1.R19 (DDR_CKP_CKAP), R7.2, R8.1
- net DDR.ODT: now reaches U4.J8 (ODT(1))
- net DDR.ODT: now also U1.L18 (DDR_ODT_NC), R10.1, R9.2
- net DDR_CKE: now reaches U4.K3 (CKE)
- net DDR_CKE: now also U1.N17 (DDR_CKE0_CKEA0), R11.2, R12.1
- net DDR.CS: now reaches U4.L3 (CS_N)
- net DDR.CS: now also U1.T20 (DDR_CS0_CSA0), R3.2, R4.1
- net at U1.K19 (DDR_ZN): now also R1.1
- new net +1V2: NT2.1
- new net +1V8: NT1.1
Other:
- title: (none) -> RAM
- moved on the sheet: U1E, U4

Commit message: more peripherals
Parts:
- C1, C2: footprint Capacitor_SMD:C_0402_1005Metric -> Capacitor_SMD:C_0201_0603Metric
- C10, C11, C12, C13, C14, C15, C16, C17, C18, C19, C20, C21, C22, C23, C24, C27, C28, C29, C30, C31, C32, C33, C34, C5, C8, C9: footprint (none) -> Capacitor_SMD:C_0201_0603Metric
- C25, C26, C3, C4, C6, C7: footprint (none) -> Capacitor_SMD:C_0402_1005Metric
- NT1: footprint (none) -> NetTie:NetTie-2_SMD_Pad0.5mm
- NT2: footprint (none) -> NetTie:NetTie-4_SMD_Pad0.5mm
- R1, R2: footprint (none) -> Resistor_SMD:R_0201_0603Metric
- R10, R11, R12, R13, R14, R15, R16, R17, R18, R19, R20, R21, R22, R23, R24, R25, R26, R27, R28, R29, R3, R30, R31, R32, R33, R34, R35, R36, R4, R5, R6, R7, R8, R9: footprint PCM_Resistor_SMD_AKL:R_0402_1005Metric -> Resistor_SMD:R_0201_0603Metric
